Commit message: Update nsra2.urdf.xacro

File: robot_ws/src/robot_descriptions/nsra2/urdf/nsra2.urdf.xacro (robot description, xacro)
@@ -14,5 +14,5 @@
   </gazebo>
   <xacro:nsra2 parent="world" prefix="$(arg prefix)">
-    <origin xyz="0 0 0" rpy="0 0 0" />
+    <origin xyz="0.220772 -0.475604 0.5" rpy="1.5708 0 3.1415" />
   </xacro:nsra2>
   <xacro:nsra2_system_position

Commit message: hough circle

File: robot_ws/src/robot_descriptions/nsra2/urdf/nsra2.urdf.xacro (robot description, xacro)
@@ -14,5 +14,5 @@
   </gazebo>
   <xacro:nsra2 parent="world" prefix="$(arg prefix)">
-    <origin xyz="0.220772 -0.475604 0.5" rpy="1.5708 0 3.1415" />
+    <origin xyz="-0.47 0.27 0.38" rpy="1.5708 0 0" />
   </xacro:nsra2>
   <xacro:nsra2_system_position

File: robot_ws/src/robot_descriptions/nsra2/urdf/nsra2_system_position.urdf.xacro (robot description, xacro)
@@ -19,5 +19,5 @@
   </gazebo>
   <xacro:nsra2 parent="world" prefix="$(arg prefix)">
-    <origin xyz="0.220772 -0.475604 0.5" rpy="1.5708 0 3.1415" />
+    <origin xyz="-0.47 0.27 0.38" rpy="1.5708 0 0" />
   </xacro:nsra2>
   <xacro:nsra2_system_position
